File: in_channel.sch (KiCad schematic (older format))
At the start: 7 parts, among them J3 PWR_IN, U3 MOC3063M, U4 LTV-814

Commit message: Finish first rev
Changed lines of the file:
@@
 EESchema Schematic File Version 4
+LIBS:230v-input-cache
 EELAYER 26 0
 EELAYER END
@@
 AR Path="/5B87BDA6/5B87B5FA" Ref="U7"  Part="1"
 AR Path="/5B87BDAA/5B87B5FA" Ref="U9"  Part="1"
-F 0 "U9" H 3015 2115 50  0000 C CNN
+F 0 "U3" H 3015 2115 50  0000 C CNN
 F 1 "MOC3063M" H 3015 2024 50  0000 C CNN
 F 2 "Housings_DIP:DIP-6_W7.62mm" H 2815 1590 50  0001 L CIN
@@
 AR Path="/5B87BDA6/5B87B601" Ref="D4"  Part="1"
 AR Path="/5B87BDAA/5B87B601" Ref="D5"  Part="1"
-F 0 "D5" H 2405 1474 50  0000 C CNN
+F 0 "D2" H 2405 1474 50  0000 C CNN
 F 1 "AL5809-15" H 2405 1565 50  0000 C CNN
 F 2 "Diodes_SMD:D_PowerDI-123" H 2405 1690 50  0001 C CNN
@@
 AR Path="/5B87BDA6/5B87B60B" Ref="U8"  Part="1"
 AR Path="/5B87BDAA/5B87B60B" Ref="U10"  Part="1"
-F 0 "U10" H 3015 2168 50  0000 C CNN
+F 0 "U4" H 3015 2168 50  0000 C CNN
 F 1 "LTV-814" H 3015 2259 50  0000 C CNN
 F 2 "Housings_DIP:DIP-4_W7.62mm" H 2815 2285 50  0001 L CIN
@@
 AR Path="/5B87BDA6/5B87B612" Ref="R11"  Part="1"
 AR Path="/5B87BDAA/5B87B612" Ref="R14"  Part="1"
-F 0 "R14" V 3288 2585 50  0000 C CNN
+F 0 "R5" V 3288 2585 50  0000 C CNN
 F 1 "12k/1W" V 3379 2585 50  0000 C CNN
 F 2 "Resistors_SMD:R_2512" V 3425 2585 50  0001 C CNN
@@
 AR Path="/5B87BDA6/5B87B619" Ref="R12"  Part="1"
 AR Path="/5B87BDAA/5B87B619" Ref="R15"  Part="1"
-F 0 "R15" H 3800 2216 50  0000 L CNN
+F 0 "R6" H 3800 2216 50  0000 L CNN
 F 1 "12k/1W" H 3800 2125 50  0000 L CNN
 F 2 "Resistors_SMD:R_2512" V 3660 2170 50  0001 C CNN
@@
 AR Path="/5B87BDA6/5B87B624" Ref="J5"  Part="1"
 AR Path="/5B87BDAA/5B87B624" Ref="J6"  Part="1"
-F 0 "J6" H 3977 1670 50  0000 R CNN
+F 0 "J3" H 3977 1670 50  0000 R CNN
 F 1 "PWR_IN" H 3977 1761 50  0000 R CNN
 F 2 "Connectors_Phoenix:PhoenixContact_MC-G_02x5.08mm_Angled" H 4005 1790 50  0001 C CNN
@@
 AR Path="/5B87BDA6/5B87B62B" Ref="#PWR0120"  Part="1"
 AR Path="/5B87BDAA/5B87B62B" Ref="#PWR0122"  Part="1"
-F 0 "#PWR0122" H 2430 1845 50  0001 C CNN
+F 0 "#PWR0116" H 2430 1845 50  0001 C CNN
 F 1 "GND" H 2435 1922 50  0000 C CNN
 F 2 "" H 2430 2095 50  0001 C CNN
@@
 AR Path="/5B87BDA6/5B87B636" Ref="#PWR0121"  Part="1"
 AR Path="/5B87BDAA/5B87B636" Ref="#PWR0123"  Part="1"
-F 0 "#PWR0123" H 2210 2095 50  0001 C CNN
+F 0 "#PWR0117" H 2210 2095 50  0001 C CNN
 F 1 "+5V" H 2225 2418 50  0000 C CNN
 F 2 "" H 2210 2245 50  0001 C CNN
@@
 AR Path="/5B87BDA6/5B87B63C" Ref="R10"  Part="1"
 AR Path="/5B87BDAA/5B87B63C" Ref="R13"  Part="1"
-F 0 "R13" V 2228 2585 50  0000 C CNN
+F 0 "R4" V 2228 2585 50  0000 C CNN
 F 1 "4k7" V 2319 2585 50  0000 C CNN
 F 2 "Resistors_SMD:R_0805" V 2365 2585 50  0001 C CNN

Commit message: Adapt to case
Parts:
- J3: footprint Connectors_Phoenix:PhoenixContact_MC-G_02x5.08mm_Angled -> Connectors_Phoenix:PhoenixContact_MSTBA-G_02x5.00mm_Angled
Changed lines of the file:
@@
 F 0 "J3" H 3977 1670 50  0000 R CNN
 F 1 "PWR_IN" H 3977 1761 50  0000 R CNN
-F 2 "Connectors_Phoenix:PhoenixContact_MC-G_02x5.08mm_Angled" H 4005 1790 50  0001 C CNN
+F 2 "Connectors_Phoenix:PhoenixContact_MSTBA-G_02x5.00mm_Angled" H 4005 1790 50  0001 C CNN
 F 3 "~" H 4005 1790 50  0001 C CNN
 	1    4005 1790
@@
 AR Path="/5B87BDA6/5B87B62B" Ref="#PWR0120"  Part="1"
 AR Path="/5B87BDAA/5B87B62B" Ref="#PWR0122"  Part="1"
-F 0 "#PWR0116" H 2430 1845 50  0001 C CNN
+F 0 "#PWR0122" H 2430 1845 50  0001 C CNN
 F 1 "GND" H 2435 1922 50  0000 C CNN
 F 2 "" H 2430 2095 50  0001 C CNN
@@
 AR Path="/5B87BDA6/5B87B636" Ref="#PWR0121"  Part="1"
 AR Path="/5B87BDAA/5B87B636" Ref="#PWR0123"  Part="1"
-F 0 "#PWR0117" H 2210 2095 50  0001 C CNN
+F 0 "#PWR0123" H 2210 2095 50  0001 C CNN
 F 1 "+5V" H 2225 2418 50  0000 C CNN
 F 2 "" H 2210 2245 50  0001 C CNN
