File: 230v-input.sch (KiCad schematic (older format))
At the start: 19 parts, among them J1 LOGIC_OUT, J2 DEBUG, U1 SAMC20E18A-AU, U2 AMSR-7805-NZ, Y1 8MHz

Commit message: Finish first rev
Parts:
- added C10, C9: 22pF, Capacitors_SMD:C_0603, symbol Device:C
- added D6: LED_RD, LEDs:LED_0805, symbol Device:LED
- added D7: LED_GN, LEDs:LED_0805, symbol Device:LED
- added D8: STPS3L60U, Diodes_SMD:D_SMB, symbol Device:D
- added IC1: UDN2987, Housings_SOIC:SOIC-20W_7.5x12.8mm_Pitch1.27mm, symbol udn2987:UDN2987
- added J7: UART, Pin_Headers:Pin_Header_Straight_1x04_Pitch2.54mm, symbol Connector:Conn_01x04_Female
- added R16: 10k, Resistors_SMD:R_0805, symbol Device:R
- added R17, R18: 470, Resistors_SMD:R_0805, symbol Device:R
- C1, C8: footprint (none) -> Capacitors_SMD:C_1206
- C2, C3, C4, C5: footprint (none) -> Capacitors_SMD:C_0603
- C6: value 120µF/50V -> 220µF/50V; footprint (none) -> Capacitors_THT:CP_Radial_D10.0mm_P5.00mm
- C7: footprint (none) -> Capacitors_SMD:C_1210
- D1: footprint (none) -> Diodes_SMD:D_SMC
- J1: footprint (none) -> Connectors_Phoenix:PhoenixContact_MC-G_06x3.81mm_Angled
- J2: footprint (none) -> Pin_Headers:Pin_Header_Straight_1x05_Pitch2.54mm
- L1: value NL12KTC820 -> DE1207-82; footprint (none) -> Inductors_SMD:L_12x12mm_h8mm
- R1, R2, R3: footprint (none) -> Inductors_SMD:L_0805
- RV1: footprint (none) -> Varistors:RV_Disc_D12_W7.5_P7.5
- U1: footprint TQFP32 -> Housings_QFP:TQFP-32_7x7mm_Pitch0.8mm
- U2: footprint (none) -> TO_SOT_Packages_THT:TO-220-3_Vertical
- Y1: footprint (none) -> Crystals:Crystal_HC49-U_Vertical
Connections:
- net labels added: +24V, FAULT, LV_OUT_A, LV_OUT_B, LV_OUT_C, LV_OUT_D, OUT_RST, UART_RX, UART_TX
- net labels removed: OUT_A, OUT_B, OUT_C, OUT_D
- wire segments 65 -> 107
- no-connect marks 0 -> 4
Other:
- moved on the sheet: J1

Commit message: Adapt to case
Parts:
- J1: footprint Connectors_Phoenix:PhoenixContact_MC-G_06x3.81mm_Angled -> Connectors_Phoenix:PhoenixContact_MSTBA-G_06x5.00mm_Angled
Changed lines of the file:
@@
 F 0 "J1" H 9006 2173 50  0000 C CNN
 F 1 "LOGIC_OUT" H 9006 2082 50  0000 C CNN
-F 2 "Connectors_Phoenix:PhoenixContact_MC-G_06x3.81mm_Angled" H 8900 1795 50  0001 C CNN
+F 2 "Connectors_Phoenix:PhoenixContact_MSTBA-G_06x5.00mm_Angled" H 8900 1795 50  0001 C CNN
 F 3 "~" H 8900 1795 50  0001 C CNN
 	1    8900 1795
@@
 Wire Wire Line
 	10070 3845 10150 3845
+Text HLabel 10150 3645 0    50   UnSpc ~ 0
+UART_RX
 Text HLabel 10150 3745 0    50   UnSpc ~ 0
-UART_RX
-Text HLabel 10150 3645 0    50   UnSpc ~ 0
 UART_TX
 Text HLabel 5200 2690 2    50   UnSpc ~ 0

Commit message: Rev 1
Parts:
- IC1: symbol udn2987:UDN2987 -> 230v-input-rescue:UDN2987-udn2987
Changed lines of the file:
@@
 SWDIO
 $Comp
-L udn2987:UDN2987 IC1
+L 230v-input-rescue:UDN2987-udn2987 IC1
 U 1 1 5B892C30
 P 7590 2245

Commit message: Rev.2
Parts:
- removed C10, C9: 22pF, Capacitors_SMD:C_0603, symbol Device:C
- removed C2: 100pF, Capacitors_SMD:C_0603, symbol Device:C
- removed R1: 330, Inductors_SMD:L_0805, symbol Device:R
- removed R2: 2k2, Inductors_SMD:L_0805, symbol Device:R
- removed R3: 1k, Inductors_SMD:L_0805, symbol Device:R
- removed Y1: 8MHz, Crystals:Crystal_HC49-U_Vertical, symbol Device:Crystal_Small
Connections:
- net MCU_RESET: now also J2.2 (Pin_2), U1.26 (~RESET~); no longer J2.4 (Pin_4)
- net SWDIO: now also J2.4 (Pin_4); no longer J2.2 (Pin_2)
Changed lines of the file:
@@
 Wire Wire Line
 	1630 3425 2020 3425
-Wire Wire Line
-	2020 3425 2020 3260
 $Comp
 L Device:C C3
@@
 	2550 3240 2550 4465
 $Comp
-L Device:R R1
-U 1 1 5B88673F
-P 1285 2690
-F 0 "R1" V 1078 2690 50  0000 C CNN
-F 1 "330" V 1169 2690 50  0000 C CNN
-F 2 "Inductors_SMD:L_0805" V 1215 2690 50  0001 C CNN
-F 3 "~" H 1285 2690 50  0001 C CNN
-	1    1285 2690
-	0    1    1    0
-$EndComp
-$Comp
 L atmel:SAMD20E14A-AU U1
 U 1 1 5B87E990
@@
 	1    0    0    -1
 $EndComp
-Text HLabel 1135 2690 0    50   Input ~ 0
+Text HLabel 1435 2690 0    50   Input ~ 0
 MCU_RESET
-Wire Wire Line
-	1435 2690 1490 2690
-$Comp
-L Device:R R2
-U 1 1 5B888B36
-P 1490 2900
-F 0 "R2" V 1435 2670 50  0000 L CNN
-F 1 "2k2" V 1405 2825 50  0000 L CNN
-F 2 "Inductors_SMD:L_0805" V 1420 2900 50  0001 C CNN
-F 3 "~" H 1490 2900 50  0001 C CNN
-	1    1490 2900
-	1    0    0    -1
-$EndComp
-$Comp
-L Device:C C2
-U 1 1 5B888C7C
-P 1750 2915
-F 0 "C2" V 1695 2705 50  0000 L CNN
-F 1 "100pF" V 1630 2815 50  0000 L CNN
-F 2 "Capacitors_SMD:C_0603" H 1788 2765 50  0001 C CNN
-F 3 "~" H 1750 2915 50  0001 C CNN
-	1    1750 2915
-	1    0    0    -1
-$EndComp
-Wire Wire Line
-	1490 3050 1490 3260
-Wire Wire Line
-	1750 3065 1750 3260
-Wire Wire Line
-	1750 3260 2020 3260
-Connection ~ 2020 3260
-Wire Wire Line
-	2020 3260 2020 3090
-Wire Wire Line
-	1750 3260 1490 3260
-Connection ~ 1750 3260
-Wire Wire Line
-	1490 2750 1490 2690
-Connection ~ 1490 2690
-Wire Wire Line
-	1490 2690 1750 2690
-Wire Wire Line
-	1750 2765 1750 2690
-Connection ~ 1750 2690
-Wire Wire Line
-	1750 2690 2700 2690
-$Comp
-L Device:R R3
-U 1 1 5B88CBCA
-P 5465 5420
-F 0 "R3" H 5535 5466 50  0000 L CNN
-F 1 "1k" H 5535 5375 50  0000 L CNN
-F 2 "Inductors_SMD:L_0805" V 5395 5420 50  0001 C CNN
-F 3 "~" H 5465 5420 50  0001 C CNN
-	1    5465 5420
-	1    0    0    -1
-$EndComp
-$Comp
-L power:+5V #PWR0113
-U 1 1 5B88CC89
-P 5465 5635
-F 0 "#PWR0113" H 5465 5485 50  0001 C CNN
-F 1 "+5V" H 5480 5808 50  0000 C CNN
-F 2 "" H 5465 5635 50  0001 C CNN
-F 3 "" H 5465 5635 50  0001 C CNN
-	1    5465 5635
-	-1   0    0    1
-$EndComp
-Wire Wire Line
-	5465 5635 5465 5570
-Wire Wire Line
-	5465 5270 5465 5090
-Wire Wire Line
-	5465 5090 5200 5090
-Text HLabel 5565 5090 2    50   Input ~ 0
+Text HLabel 5200 5090 2    50   Input ~ 0
 SWCLK
-Wire Wire Line
-	5465 5090 5565 5090
-Connection ~ 5465 5090
-Wire Wire Line
-	5200 5190 5565 5190
-Text HLabel 5565 5190 2    50   Input ~ 0
+Text HLabel 5200 5190 2    50   Input ~ 0
 SWDIO
-$Comp
-L Device:Crystal_Small Y1
-U 1 1 5B89178E
-P 5795 3890
-F 0 "Y1" H 5795 4115 50  0000 C CNN
-F 1 "8MHz" H 5795 4024 50  0000 C CNN
-F 2 "Crystals:Crystal_HC49-U_Vertical" H 5795 3890 50  0001 C CNN
-F 3 "~" H 5795 3890 50  0001 C CNN
-	1    5795 3890
-	1    0    0    -1
-$EndComp
-Wire Wire Line
-	5695 3890 5650 3890
-Wire Wire Line
-	5200 3990 5970 3990
-Wire Wire Line
-	5970 3990 5970 3890
-Wire Wire Line
-	5970 3890 5895 3890
 Text HLabel 10010 985  0    50   UnSpc ~ 0
 DETECT_A
@@
 Wire Wire Line
 	1375 6555 1275 6555
-Text HLabel 1275 6455 2    50   UnSpc ~ 0
+Text HLabel 1275 6255 2    50   UnSpc ~ 0
 MCU_RESET
 Text HLabel 1275 6355 2    50   UnSpc ~ 0
 SWCLK
-Text HLabel 1275 6255 2    50   UnSpc ~ 0
+Text HLabel 1275 6455 2    50   UnSpc ~ 0
 SWDIO
 $Comp
@@
 FAULT
 $Comp
-L Device:C C9
-U 1 1 5B8B4D3D
-P 6250 4095
-F 0 "C9" H 6365 4141 50  0000 L CNN
-F 1 "22pF" H 6365 4050 50  0000 L CNN
-F 2 "Capacitors_SMD:C_0603" H 6288 3945 50  0001 C CNN
-F 3 "~" H 6250 4095 50  0001 C CNN
-	1    6250 4095
-	1    0    0    -1
-$EndComp
-$Comp
-L Device:C C10
-U 1 1 5B8B4DC1
-P 6665 4105
-F 0 "C10" H 6780 4151 50  0000 L CNN
-F 1 "22pF" H 6780 4060 50  0000 L CNN
-F 2 "Capacitors_SMD:C_0603" H 6703 3955 50  0001 C CNN
-F 3 "~" H 6665 4105 50  0001 C CNN
-	1    6665 4105
-	1    0    0    -1
-$EndComp
-Wire Wire Line
-	5970 3890 6250 3890
-Wire Wire Line
-	6250 3890 6250 3945
-Connection ~ 5970 3890
-Wire Wire Line
-	5650 3800 6665 3800
-Wire Wire Line
-	6665 3800 6665 3955
-Wire Wire Line
-	5650 3800 5650 3890
-Connection ~ 5650 3890
-Wire Wire Line
-	5650 3890 5200 3890
-$Comp
-L power:GND #PWR03
-U 1 1 5B8BA3DD
-P 6465 4355
-F 0 "#PWR03" H 6465 4105 50  0001 C CNN
-F 1 "GND" H 6470 4182 50  0000 C CNN
-F 2 "" H 6465 4355 50  0001 C CNN
-F 3 "" H 6465 4355 50  0001 C CNN
-	1    6465 4355
-	1    0    0    -1
-$EndComp
-Wire Wire Line
-	6465 4355 6465 4310
-Wire Wire Line
-	6465 4310 6665 4310
-Wire Wire Line
-	6665 4310 6665 4255
-Wire Wire Line
-	6465 4310 6250 4310
-Wire Wire Line
-	6250 4310 6250 4245
-Connection ~ 6465 4310
-$Comp
 L Connector:Conn_01x04_Female J7
 U 1 1 5B8BE3CE
@@
 Wire Wire Line
 	8145 1175 8340 1175
+Wire Wire Line
+	2020 3090 2020 3425
+Wire Wire Line
+	1435 2690 2700 2690
 $EndSCHEMATC
